File: BNOCAN/_autosave-BNOCAN.kicad_pcb (KiCad board)
At the start: 2 copper layers, 46 parts, among them J1 CANConn, SW1 RST, U1 TPS560430X3FDBVR, U2 SN65HVD230, U4 STM32F103T8Ux, U5 BNO085, Y1 G43270019, Y2 STMCRYSTAL

Commit message: V1 Ordered
Parts:
- removed C13: Bulk, Capacitor_THT:CP_Radial_D8.0mm_P3.80mm
- removed C20: 100nF, Capacitor_SMD:C_0402_1005Metric
- removed R17: 56, Resistor_SMD:R_0805_2012Metric_Pad1.20x1.40mm_HandSolder
- added D3: GLED, LED_SMD:LED_0603_1608Metric, F.Cu at (136.9, 99.9)
- added H1: MountingHole, MountingHole:MountingHole_3.2mm_M3, F.Cu at (114.0, 59.2)
- added H2: MountingHole, MountingHole:MountingHole_3.2mm_M3, F.Cu at (156.1, 101.1)
- added H3: MountingHole, MountingHole:MountingHole_3.2mm_M3, F.Cu at (114.0, 101.2)
- added J2: PWRConn, Connector_Wire:SolderWire-0.15sqmm_1x02_P4mm_D0.5mm_OD1.5mm_Relief, F.Cu at (120.0, 93.1)
- added J3: SWDConn, Connector_PinHeader_1.27mm:PinHeader_2x07_P1.27mm_Vertical_SMD, F.Cu at (151.1, 63.7)
- added JP1: CANjp, Connector_PinHeader_2.54mm:PinHeader_1x02_P2.54mm_Vertical, F.Cu at (145.9, 84.0)
- added Q1: MMBT3904, Package_TO_SOT_SMD:SOT-23, F.Cu at (133.6, 93.0)
- added Q2: MMBT3904, Package_TO_SOT_SMD:SOT-23, F.Cu at (138.0, 93.0)
- added R18: 100, Resistor_SMD:R_0402_1005Metric, F.Cu at (136.4, 90.6)
- added R3: 100, Resistor_SMD:R_0402_1005Metric, F.Cu at (132.6, 95.9)
- added R4: 100, Resistor_SMD:R_0402_1005Metric, F.Cu at (137.1, 95.9)
- added R5: 100, Resistor_SMD:R_0402_1005Metric, F.Cu at (132.2, 90.5)
- C11, C12, C5, C6: footprint Capacitor_SMD:C_0805_2012Metric -> Capacitor_SMD:C_0402_1005Metric
- C15: footprint Resistor_SMD:R_0603_1608Metric -> Capacitor_SMD:C_0603_1608Metric
- C3: footprint Capacitor_SMD:C_0603_1608Metric -> Capacitor_SMD:C_0402_1005Metric
- C9: footprint Capacitor_SMD:C_0402_1005Metric -> Capacitor_SMD:C_0603_1608Metric
- D1: value SK6812 -> RLED; footprint LED_SMD:LED_SK6812_PLCC4_5.0x5.0mm_P3.2mm -> LED_SMD:LED_0603_1608Metric
- J1: footprint Connector_Wire:SolderWire-1.5sqmm_1x02_P7.8mm_D1.7mm_OD3.9mm_Relief -> Connector_Wire:SolderWire-0.15sqmm_1x02_P4mm_D0.5mm_OD1.5mm_Relief
- R16: value 56 -> 120
- moved C1 169.4 mm to (151.4, 78.4)
- moved J1 160.1 mm to (145.9, 93.1)
- moved C7 159.9 mm to (139.1, 83.0), turned to -90 degrees
- moved C8 158.3 mm to (136.6, 86.0)
- moved C9 158.1 mm to (136.7, 87.3)
- moved C18 152.8 mm to (140.9, 71.9), turned to -90 degrees
- moved C17 152.4 mm to (142.8, 65.1), turned to 90 degrees
- moved C16 143.5 mm to (131.8, 65.4), turned to 90 degrees
- moved C14 143.5 mm to (131.5, 67.8)
- moved C19 142.5 mm to (131.5, 69.5), turned to 180 degrees
- moved D2 113.0 mm to (151.4, 89.1), turned to -90 degrees
- moved R15 108.3 mm to (155.3, 86.2), turned to 90 degrees
- moved U2 94.8 mm to (151.4, 82.9), turned to -90 degrees
- moved D1 94.5 mm to (133.7, 99.9), turned to 90 degrees
- moved C15 92.0 mm to (141.0, 64.6), turned to 90 degrees
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Connections:
- net Net-(U4-NRST) renamed /~{RST}
- D1 pad 2: Net-(D1-DIN) -> Net-(D1-A)
- J1 pad 1: /CAN+ -> /CAN-
- J1 pad 2: /CAN- -> /CAN+
- R1 pad 1: Net-(U1-SW) -> +3.3V
- U4 pad 10: unconnected-(U4-PA3-Pad10) -> Net-(U4-PA3)
- U4 pad 16: /ProtocolSel1 -> /ProtocolSel0
- U4 pad 17: /ProtocolSel0 -> /ProtocolSel1
- U4 pad 9: Net-(D1-DIN) -> Net-(U4-PA2)
- U5 pad 26: (no net) -> Net-(U5-CLKSEL1/XOUT32)
Routing:
- net +3.3V: track 0.00 -> 201.1 mm, vias 0 -> 3
- net Net-(U4-BOOT0): track 0.00 -> 44.9 mm, vias 0 -> 2
- net /~{RST}: track 0.00 -> 40.3 mm
- net Net-(U4-PA3): track 0.00 -> 28.1 mm
- net Net-(U4-PA2): track 0.00 -> 24.4 mm
- net /ProtocolSel1: track 0.00 -> 21.2 mm
- net /ProtocolSel0: track 0.00 -> 18.8 mm
- net /CAN-: track 0.00 -> 18.5 mm
- net /CAN_RX: track 0.00 -> 18.0 mm
- net /CAN+: track 0.00 -> 18.0 mm
- net Net-(U4-PA9): track 0.00 -> 17.8 mm, vias 0 -> 2
- net /CAN_TX: track 0.00 -> 16.1 mm
- net /UART_RX: track 0.00 -> 15.3 mm, vias 0 -> 2
- net /SWO: track 0.00 -> 15.1 mm
- net /SWCLK: track 0.00 -> 13.4 mm
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- added copper zone on B.Cu, net GND
- added copper zone on F.Cu, net GND
- added copper zone on F.Cu, net VCC
Other:
- board outline added: 50 x 50 mm
- board text added: "+ - PWR [4-36V]"
- board text added: "BNOCAN Raheel Rehmatullah December 2023"
- board text added: "BOOT"
- board text added: "CAN L H"
- board text added: "CAN TERM"
- board text added: "DEBUG"
