File: BNOCAN/BNOCAN.kicad_sch (KiCad schematic)
At the start: 56 parts, among them J1 CANConn, J2 PWRConn, J3 SWDConn, Q1 MMBT3904, Q2 MMBT3904, SW1 RST, U1 TPS560430X3FDBVR, U2 SN65HVD230, U4 STM32F103T8Ux, U5 BNO085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

Commit message: V1.1 Produced
Parts:
- removed C21: Super, Capacitor_THT:CP_Radial_D13.0mm_P5.00mm, symbol Device:C_Polarized_Small
- removed Q1, Q2: MMBT3904, Package_TO_SOT_SMD:SOT-23, symbol Transistor_BJT:MMBT3904
- removed R1: 51k, Resistor_SMD:R_0603_1608Metric, symbol Device:R_Small
- removed R18, R3: 100, Resistor_SMD:R_0402_1005Metric, symbol Device:R_Small
- removed R2: 22.1k, Resistor_SMD:R_0603_1608Metric, symbol Device:R_Small
- removed R6, R7, R8: 0, Resistor_SMD:R_0402_1005Metric, symbol Device:R_Small
- added R17: 10k, Resistor_SMD:R_0603_1608Metric, symbol Device:R_Small
- C11, C12, Y2: now fitted
- SW1: value RST -> BOOT
Connections:
- net ~{RST} is gone; now on net ~{NRST}: C14.2, J3.12 (Pin_12), U4.4 (NRST)
- net +3.3V: now also C10.1, SW1.2, U1.3 (FB), R17.1; no longer R14.2, U5.4 (BOOTN)
- net GND: now also R14.2; no longer C10.2, SW1.1
- net MISO: now also U5.20 (H_SDA/MISO/TX)
- net MOSI: now also U5.17 (H_SA0/MOSI)
- net SPICLK: now also U5.19 (H_SCL/SCLK/RX)
- net ~{IMU_INTR}: now also U4.20 (PA8)
- net at U4.10 (PA3): now also R4.2
- net ~{CS}: now reaches U4.11 (PA4)
- net ~{CS}: now also U5.18 (H_CSN)
- net at R14.1, U4.35 (BOOT0): now also C10.2, SW1.1; no longer C10.1, SW1.2
- net at R5.2: now also D1.2 (A)
- net NRST renamed ~{NRST}
- new net: R17.2, U5.4 (BOOTN)
- no-connect marks 11 -> 10
Other:
- note added: "-C4 Rated for 10V -inductor rating see table 1 in IC datasheet -VREF = 1V -Note, if you are recreating this design for your power supply, it references the WEBENCH generated schematic as opposed to the datasheet schematic, which was incorrect in my case (I only saw VCC-Vref on output with the datasheet schematic)"
- note added: "TODO/CHANGELOG [DONE]-FIX BOOT SET HIGH (SHOULD BE LOW) [DONE]-FIX BNO085 RST [DONE]-FIX BUCK CONVERTER FEEDBACK CIRCUIT [DONE]-ADD ~{IMUINTR} to MCU [DONE]-REMOVE LED TRANSISTORS -REVERSE POLARITY PROTECTION -ADD STM32 CRYSTAL TO INCREASE CANBUS STABILITY"
- note removed: "-C4 Rated for 10V -inductor rating see table 1 in IC datasheet -VREF = 1V"
- moved on the sheet: C10, D1, D3, L1, R12, R13, R14, R4, SW1

Commit message: Firmware Dump + some Board Bug fixes
Parts:
- removed Y2: STMCRYSTAL, Crystal:Crystal_SMD_3215-2Pin_3.2x1.5mm, symbol Device:Crystal
- added Y2: STMCRYSTAL, Crystal:Crystal_SMD_3225-4Pin_3.2x2.5mm, symbol Device:Crystal_GND24
- C11, C12: value 22pF -> 8pF
- R14: footprint Capacitor_SMD:C_0603_1608Metric -> Resistor_SMD:R_0603_1608Metric
Connections:
- net GND: now also Y2.2, Y2.4
- net at C12.1, U4.2 (PD0): now also Y2.3
- net at C11.1, U4.3 (PD1): now also Y2.1
Other:
- note added: "TODO/CHANGELOG [DONE]-FIX BOOT SET HIGH (SHOULD BE LOW) [DONE]-FIX BNO085 RST [DONE]-FIX BUCK CONVERTER FEEDBACK CIRCUIT [DONE]-ADD ~{IMUINTR} to MCU [DONE]-REMOVE LED TRANSISTORS [DONE]-Fixed STMCRYSTAL -REVERSE POLARITY PROTECTION -ADD STM32 CRYSTAL TO INCREASE CANBUS STABILITY"
- note removed: "TODO/CHANGELOG [DONE]-FIX BOOT SET HIGH (SHOULD BE LOW) [DONE]-FIX BNO085 RST [DONE]-FIX BUCK CONVERTER FEEDBACK CIRCUIT [DONE]-ADD ~{IMUINTR} to MCU [DONE]-REMOVE LED TRANSISTORS -REVERSE POLARITY PROTECTION -ADD STM32 CRYSTAL TO INCREASE CANBUS STABILITY"
Changed lines of the file:
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@@
 	)
 	(junction
+		(at 76.2 153.67)
+		(diameter 0)
+		(color 0 0 0 0)
+	)
+	(junction
 		(at 81.28 147.32)
 		(diameter 0)
@@
 	)
 	(junction
+		(at 66.04 153.67)
+		(diameter 0)
+		(color 0 0 0 0)
+	)
+	(junction
 		(at 254 64.77)
 		(diameter 0)
@@
 	(wire
 		(pts
+			(xy 76.2 153.67) (xy 86.36 153.67)
+		)
+		(stroke
+			(width 0)
+			(type default)
+		)
+	)
+	(wire
+		(pts
 			(xy 123.19 137.16) (xy 124.46 137.16)
 		)
@@
 	(wire
 		(pts
-			(xy 66.04 160.02) (xy 66.04 147.32)
+			(xy 66.04 153.67) (xy 66.04 147.32)
+		)
+		(stroke
+			(width 0)
+			(type default)
+		)
+	)
+	(wire
+		(pts
+			(xy 66.04 160.02) (xy 66.04 153.67)
 		)
 		(stroke
@@
 	(wire
 		(pts
+			(xy 66.04 153.67) (xy 76.2 153.67)
+		)
+		(stroke
+			(width 0)
+			(type default)
+		)
+	)
+	(wire
+		(pts
 			(xy 124.46 190.5) (xy 124.46 189.23)
 		)
@@
 		)
 	)
-	(text "TODO/CHANGELOG\n[DONE]-FIX BOOT SET HIGH (SHOULD BE LOW) \n[DONE]-FIX BNO085 RST \n[DONE]-FIX BUCK CONVERTER FEEDBACK CIRCUIT \n[DONE]-ADD ~{IMUINTR} to MCU \n[DONE]-REMOVE LED TRANSISTORS\n-REVERSE POLARITY PROTECTION\n-ADD STM32 CRYSTAL TO INCREASE CANBUS STABILITY\n\n"
+	(text "TODO/CHANGELOG\n[DONE]-FIX BOOT SET HIGH (SHOULD BE LOW) \n[DONE]-FIX BNO085 RST \n[DONE]-FIX BUCK CONVERTER FEEDBACK CIRCUIT \n[DONE]-ADD ~{IMUINTR} to MCU \n[DONE]-REMOVE LED TRANSISTORS\n[DONE]-Fixed STMCRYSTAL\n-REVERSE POLARITY PROTECTION\n-ADD STM32 CRYSTAL TO INCREASE CANBUS STABILITY\n\n"
 		(exclude_from_sim no)
 		(at 50.8 195.58 0)
@@
 			)
 		)
-		(property "Footprint" "Capacitor_SMD:C_0603_1608Metric"
+		(property "Footprint" "Resistor_SMD:R_0603_1608Metric"
 			(at 73.66 129.54 0)
 			(effects
@@
 			)
 		)
-		(property "Value" "22pF"
+		(property "Value" "8pF"
 			(at 73.6536 143.51 90)
 			(effects
@@
 		(on_board yes)
 		(dnp no)
-		(fields_autoplaced yes)
 		(property "Reference" "C11"
-			(at 73.6537 166.37 90)
+			(at 73.66 163.83 90)
 			(effects
 				(font
@@
 			)
 		)
-		(property "Value" "22pF"
-			(at 73.6537 163.83 90)
+		(property "Value" "8pF"
+			(at 73.66 166.37 90)
 			(effects
 				(font
@@
 	)
 	(symbol
-		(lib_id "Device:Crystal")
-		(at 81.28 153.67 270)
+		(lib_id "Device:R_Small")
+		(at 160.02 124.46 0)
 		(unit 1)
 		(exclude_from_sim no)
@@
 		(on_board yes)
 		(dnp no)
-		(property "Reference" "Y2"
-			(at 76.2 152.4 90)
+		(property "Reference" "R4"
+			(at 157.48 123.19 90)
 			(effects
 				(font
 					(size 1.27 1.27)
 				)
-				(justify left)
 			)
 		)
-		(property "Value" "STMCRYSTAL"
-			(at 67.31 154.94 90)
+		(property "Value" "100"
+			(at 157.48 127 90)
 			(effects
 				(font
 					(size 1.27 1.27)
 				)
-				(justify left)
 			)
 		)
-		(property "Footprint" "Crystal:Crystal_SMD_3215-2Pin_3.2x1.5mm"
-			(at 81.28 153.67 0)
+		(property "Footprint" "Resistor_SMD:R_0402_1005Metric"
+			(at 160.02 124.46 0)
 			(effects
 				(font
@@
 		)
 		(property "Datasheet" "~"
-			(at 81.28 153.67 0)
+			(at 160.02 124.46 0)
 			(effects
 				(font
@@
 		)
 		(property "Description" ""
-			(at 81.28 153.67 0)
+			(at 160.02 124.46 0)
 			(effects
 				(font
@@
 			(project "BNOCAN"
 				(path "/ac9e7a91-5467-4281-9ed7-cf1345349504"
-					(reference "Y2")
+					(reference "R4")
 					(unit 1)
 				)
@@
 	(symbol
 		(lib_id "Device:R_Small")
-		(at 160.02 124.46 0)
+		(at 181.61 58.42 90)
 		(unit 1)
 		(exclude_from_sim no)
@@
 		(on_board yes)
 		(dnp no)
-		(property "Reference" "R4"
-			(at 157.48 123.19 90)
+		(property "Reference" "R17"
+			(at 181.61 60.96 90)
 			(effects
 				(font
@@
 			)
 		)
-		(property "Value" "100"
-			(at 157.48 127 90)
+		(property "Value" "10k"
+			(at 181.61 55.88 90)
 			(effects
 				(font
@@
 			)
 		)
-		(property "Footprint" "Resistor_SMD:R_0402_1005Metric"
-			(at 160.02 124.46 0)
+		(property "Footprint" "Resistor_SMD:R_0603_1608Metric"
+			(at 181.61 58.42 0)
 			(effects
 				(font
@@
 		)
 		(property "Datasheet" "~"
-			(at 160.02 124.46 0)
+			(at 181.61 58.42 0)
 			(effects
 				(font
@@
 		)
 		(property "Description" ""
-			(at 160.02 124.46 0)
+			(at 181.61 58.42 0)
 			(effects
 				(font
@@
 			(project "BNOCAN"
 				(path "/ac9e7a91-5467-4281-9ed7-cf1345349504"
-					(reference "R4")
+					(reference "R17")
 					(unit 1)
 				)
@@
 	)
 	(symbol
-		(lib_id "Device:R_Small")
-		(at 181.61 58.42 90)
+		(lib_id "Device:Crystal_GND24")
+		(at 81.28 153.67 90)
 		(unit 1)
 		(exclude_from_sim no)
@@
 		(on_board yes)
 		(dnp no)
-		(property "Reference" "R17"
-			(at 181.61 60.96 90)
+		(property "Reference" "Y2"
+			(at 83.566 142.494 90)
 			(effects
 				(font
@@
 			)
 		)
-		(property "Value" "10k"
-			(at 181.61 55.88 90)
+		(property "Value" "STMCRYSTAL"
+			(at 83.566 145.034 90)
 			(effects
 				(font
@@
 			)
 		)
-		(property "Footprint" "Resistor_SMD:R_0603_1608Metric"
-			(at 181.61 58.42 0)
+		(property "Footprint" "Crystal:Crystal_SMD_3225-4Pin_3.2x2.5mm"
+			(at 81.28 153.67 0)
 			(effects
 				(font
@@
 		)
 		(property "Datasheet" "~"
-			(at 181.61 58.42 0)
+			(at 81.28 153.67 0)
 			(effects
 				(font
@@
 			)
 		)
-		(property "Description" ""
-			(at 181.61 58.42 0)
+		(property "Description" "Four pin crystal, GND on pins 2 and 4"
+			(at 81.28 153.67 0)
 			(effects
 				(font
@@
 			)
 		)
-		(pin "1"
+		(pin "3"
 		)
 		(pin "2"
 		)
+		(pin "1"
+		)
+		(pin "4"
+		)
 		(instances
 			(project "BNOCAN"
 				(path "/ac9e7a91-5467-4281-9ed7-cf1345349504"
-					(reference "R17")
+					(reference "Y2")
 					(unit 1)
 				)
